File: ignitor.sch (EAGLE design)
At the start: 80 parts, among them IC1 T2333, IC2 TA80005, IC3 D131850-0760, T1 B647, T2 C945, T3 1005, T4 MJE801, T5 1005, T6 MJE801, U1 ATMEGA48-20PU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

Commit message: Memory keep
Parts:
- added _C1, _C2: 22p, resistor:C-EUC0805
- X1: value 12.07 MHz -> 20 MHz
Connections:
- net EXTAL: now also X1.1, _C1.2; no longer X1.3
- net GND: now also _C1.1, _C2.1
- net XTAL: now also X1.3, _C2.2; no longer X1.1
Other:
- moved on the sheet: C14, C16, R15, R17, X1

Commit message: Fixed parser
Parts:
- added LED1: (no value), led:LED3MM
Connections:
- removed net N$44: IC3.37, R21.1
- new net LED: IC3.37, LED1.A, R21.1
- new net N$7: LED1.C, U1.PD4
- net GND: no longer U1.PD4
Changed lines of the file:
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@@
 <?xml version="1.0" encoding="utf-8"?>
 <!DOCTYPE eagle SYSTEM "eagle.dtd">
-<eagle version="7.6.0">
+<eagle version="7.2.0">
 <drawing>
 <settings>
@@
 <part name="_C2" library="resistor" deviceset="C-EU" device="C0805" value="22p"/>
 <part name="_C1" library="resistor" deviceset="C-EU" device="C0805" value="22p"/>
+<part name="LED1" library="led" deviceset="LED" device="3MM"/>
 </parts>
 <sheets>
@@
 <instance part="_C2" gate="G$1" x="208.28" y="99.06" rot="MR180"/>
 <instance part="_C1" gate="G$1" x="198.12" y="99.06" rot="MR180"/>
+<instance part="LED1" gate="G$1" x="264.16" y="160.02" rot="R180"/>
 </instances>
 <busses>
@@
 <segment>
 <pinref part="GND29" gate="1" pin="GND"/>
-<pinref part="U1" gate="A" pin="PD4"/>
-<wire x1="246.38" y1="172.72" x2="248.92" y2="172.72" width="0.1524" layer="91"/>
-<wire x1="248.92" y1="172.72" x2="248.92" y2="165.1" width="0.1524" layer="91"/>
 <wire x1="248.92" y1="165.1" x2="254" y2="165.1" width="0.1524" layer="91"/>
 <wire x1="254" y1="165.1" x2="254" y2="162.56" width="0.1524" layer="91"/>
-<junction x="248.92" y="172.72"/>
 <pinref part="U1" gate="A" pin="PC5"/>
 <wire x1="246.38" y1="190.5" x2="248.92" y2="190.5" width="0.1524" layer="91"/>
-<wire x1="248.92" y1="190.5" x2="248.92" y2="172.72" width="0.1524" layer="91"/>
+<wire x1="248.92" y1="190.5" x2="248.92" y2="165.1" width="0.1524" layer="91"/>
 <pinref part="U1" gate="A" pin="PC4"/>
 <wire x1="246.38" y1="193.04" x2="248.92" y2="193.04" width="0.1524" layer="91"/>
@@
 </segment>
 </net>
-<net name="N$44" class="0">
-<segment>
+<net name="LED" class="0">
+<segment>
+<pinref part="R21" gate="G$1" pin="1"/>
+<wire x1="271.78" y1="83.82" x2="271.78" y2="86.36" width="0.1524" layer="91"/>
 <pinref part="IC3" gate="G$1" pin="37"/>
-<pinref part="R21" gate="G$1" pin="1"/>
-<wire x1="251.46" y1="83.82" x2="271.78" y2="83.82" width="0.1524" layer="91"/>
-<wire x1="271.78" y1="83.82" x2="271.78" y2="86.36" width="0.1524" layer="91"/>
+<wire x1="271.78" y1="83.82" x2="251.46" y2="83.82" width="0.1524" layer="91"/>
+<label x="254" y="84.328" size="1.27" layer="95"/>
+</segment>
+<segment>
+<pinref part="LED1" gate="G$1" pin="A"/>
+<wire x1="264.16" y1="157.48" x2="264.16" y2="152.4" width="0.1524" layer="91"/>
 </segment>
 </net>
@@
 </segment>
 </net>
+<net name="N$7" class="0">
+<segment>
+<pinref part="U1" gate="A" pin="PD4"/>
+<wire x1="246.38" y1="172.72" x2="264.16" y2="172.72" width="0.1524" layer="91"/>
+<wire x1="264.16" y1="172.72" x2="264.16" y2="165.1" width="0.1524" layer="91"/>
+<pinref part="LED1" gate="G$1" pin="C"/>
+</segment>
+</net>
