File: board/ignitor.sch (EAGLE design)
At the start: 83 parts, among them IC1 T2333, IC2 TA80005, IC3 D131850-0760, T1 B647, T2 C945, T3 1005, T4 MJE801, T5 1005, T6 MJE801, U1 ATMEGA48-20PU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

Commit message: Project updated
Connections:
- net COIL_BACK renamed COIL_REAR
- new net !IGN_REAR: IC3.9, R22.2, T2.B
- net !IGN_BACK: no longer IC3.9, R22.2, T2.B
Changed lines of the file:
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@@
 <?xml version="1.0" encoding="utf-8"?>
 <!DOCTYPE eagle SYSTEM "eagle.dtd">
-<eagle version="7.2.0">
+<eagle version="7.6.0">
 <drawing>
 <settings>
@@
 <setting verticaltext="up"/>
 </settings>
-<grid distance="0.1" unitdist="inch" unit="inch" style="lines" multiple="1" display="yes" altdistance="0.01" altunitdist="inch" altunit="inch"/>
+<grid distance="0.1" unitdist="inch" unit="inch" style="lines" multiple="1" display="no" altdistance="0.01" altunitdist="inch" altunit="inch"/>
 <layers>
 <layer number="1" name="Top" color="4" fill="1" visible="no" active="no"/>
@@
 </segment>
 </net>
-<net name="COIL_BACK" class="0">
+<net name="COIL_REAR" class="0">
 <segment>
 <pinref part="SV1" gate="1" pin="2"/>
@@
 </net>
 <net name="!IGN_BACK" class="0">
-<segment>
-<pinref part="T2" gate="G$1" pin="B"/>
-<wire x1="96.52" y1="25.4" x2="109.22" y2="25.4" width="0.1524" layer="91"/>
-<pinref part="IC3" gate="G$1" pin="9"/>
-<wire x1="109.22" y1="25.4" x2="175.26" y2="25.4" width="0.1524" layer="91"/>
-<wire x1="175.26" y1="25.4" x2="175.26" y2="71.12" width="0.1524" layer="91"/>
-<wire x1="175.26" y1="71.12" x2="236.22" y2="71.12" width="0.1524" layer="91"/>
-<pinref part="R22" gate="G$1" pin="2"/>
-<wire x1="109.22" y1="27.94" x2="109.22" y2="25.4" width="0.1524" layer="91"/>
-<junction x="109.22" y="25.4"/>
-<label x="223.52" y="71.628" size="1.27" layer="95"/>
-</segment>
 <segment>
 <pinref part="U1" gate="A" pin="PC3"/>
@@
 </segment>
 </net>
+<net name="!IGN_REAR" class="0">
+<segment>
+<pinref part="T2" gate="G$1" pin="B"/>
+<wire x1="96.52" y1="25.4" x2="109.22" y2="25.4" width="0.1524" layer="91"/>
+<pinref part="IC3" gate="G$1" pin="9"/>
+<wire x1="109.22" y1="25.4" x2="175.26" y2="25.4" width="0.1524" layer="91"/>
+<wire x1="175.26" y1="25.4" x2="175.26" y2="71.12" width="0.1524" layer="91"/>
+<wire x1="175.26" y1="71.12" x2="236.22" y2="71.12" width="0.1524" layer="91"/>
+<pinref part="R22" gate="G$1" pin="2"/>
+<wire x1="109.22" y1="27.94" x2="109.22" y2="25.4" width="0.1524" layer="91"/>
+<junction x="109.22" y="25.4"/>
+<label x="223.52" y="71.628" size="1.27" layer="95"/>
+</segment>
+</net>
